File: BubblerMain/BubblerMain.kicad_pcb (KiCad board)
At the start: 4 copper layers, 72 x 66 mm, 85 parts, among them J1 Conn_01x04_Pin, J10 Conn_01x04_Pin, J11 Conn_01x08_Pin, J12 Conn_01x08_Pin, J2 Conn_01x03_Pin, J3 Conn_01x03_Pin, J4 Conn_01x03_Pin, J5 Conn_01x03_Pin, J6 Conn_01x02_Pin, J7 Conn_01x02_Pin, J8 USB_C_Receptacle, J9 Conn_01x08_Pin, Q1 DMP3013SFV, SW1 SW_Push, SW2 SW_Push, SW3 LED, U1 74AHCT125, U3 TPS563201DDCR, U4 ESP32-S3-WROOM-1, U5 AP2112K-3.3, U6 USBLC6-2SC6, U7 THVD1400D, U8 SM712, U9 TPS565201DDCR

Commit message: annotations
Connections:
- J12 pad 1: GND1 -> unconnected-(J12-Pin_1-Pad1)
Routing:
- net +5V: track 170.4 -> 79.8 mm
- net +3V3: track 193.8 -> 186.4 mm
- net LED1 Signal: track 66.7 -> 68.7 mm
- net Net-(R9-Pad2): track 16.6 -> 15.0 mm
- added copper zone on In2.Cu, net +3V3
- added copper zone on In2.Cu, net Net-(J6-Pin_2)
Other:
- board text added: "MilaTotem v1.1"
- board text removed: "MilaTotem v1.0"
