File: BubblerMain/esp32_module.kicad_sch (KiCad schematic)
At the start: 31 parts, among them J12 Conn_01x08_Pin, J8 USB_C_Receptacle, J9 Conn_01x08_Pin, SW1 SW_Push, SW2 SW_Push, SW3 LED, U4 ESP32-S3-WROOM-1, U5 AP2112K-3.3, U6 USBLC6-2SC6

Commit message: BubblerRemote initial commit
Connections:
- net GND1: no longer J12.1 (Pin_1)
Other:
- moved on the sheet: J12
Changed lines of the file:
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@@
 	(wire
 		(pts
-			(xy 59.69 176.53) (xy 59.69 172.72)
-		)
-		(stroke
-			(width 0)
-			(type default)
-		)
-	)
-	(wire
-		(pts
-			(xy 39.37 167.64) (xy 49.53 167.64)
+			(xy 41.91 190.5) (xy 82.55 190.5)
 		)
 		(stroke
@@
 	(wire
 		(pts
-			(xy 39.37 180.34) (xy 63.5 180.34)
+			(xy 41.91 177.8) (xy 90.17 177.8)
 		)
 		(stroke
@@
 	(wire
 		(pts
-			(xy 46.99 187.96) (xy 53.34 187.96)
+			(xy 49.53 168.91) (xy 90.17 168.91)
 		)
 		(stroke
@@
 	(wire
 		(pts
-			(xy 58.42 176.53) (xy 58.42 177.8)
-		)
-		(stroke
-			(width 0)
-			(type default)
-		)
-	)
-	(wire
-		(pts
 			(xy 266.7 19.05) (xy 265.43 19.05)
 		)
@@
 	(wire
 		(pts
-			(xy 49.53 167.64) (xy 49.53 168.91)
-		)
-		(stroke
-			(width 0)
-			(type default)
-		)
-	)
-	(wire
-		(pts
 			(xy 22.86 46.99) (xy 22.86 52.07)
 		)
@@
 	(wire
 		(pts
-			(xy 58.42 176.53) (xy 59.69 176.53)
-		)
-		(stroke
-			(width 0)
-			(type default)
-		)
-	)
-	(wire
-		(pts
 			(xy 81.28 74.93) (xy 120.65 74.93)
 		)
@@
 	(wire
 		(pts
-			(xy 58.42 177.8) (xy 39.37 177.8)
+			(xy 41.91 180.34) (xy 68.58 180.34)
 		)
 		(stroke
@@
 	(wire
 		(pts
-			(xy 39.37 167.64) (xy 39.37 175.26)
+			(xy 41.91 190.5) (xy 41.91 185.42)
 		)
 		(stroke
@@
 	(wire
 		(pts
-			(xy 46.99 182.88) (xy 46.99 187.96)
+			(xy 49.53 175.26) (xy 49.53 168.91)
 		)
 		(stroke
@@
 	(wire
 		(pts
-			(xy 39.37 182.88) (xy 46.99 182.88)
+			(xy 41.91 175.26) (xy 49.53 175.26)
 		)
 		(stroke
@@
 	(global_label "Motor Power"
 		(shape output)
-		(at 59.69 172.72 0)
+		(at 68.58 180.34 0)
 		(fields_autoplaced yes)
 		(effects
@@
 		)
 		(property "Intersheetrefs" "${INTERSHEET_REFS}"
-			(at 74.5284 172.72 0)
+			(at 83.4184 180.34 0)
 			(effects
 				(font
@@
 	(symbol
 		(lib_id "Connector:Conn_01x04_Pin")
-		(at 34.29 177.8 0)
+		(at 36.83 180.34 0)
+		(mirror x)
 		(unit 1)
 		(exclude_from_sim no)
@@
 		(on_board yes)
 		(dnp no)
-		(fields_autoplaced yes)
 		(property "Reference" "J12"
-			(at 34.925 170.18 0)
+			(at 37.465 187.96 0)
 			(effects
 				(font
@@
 		)
 		(property "Value" "Conn_01x08_Pin"
-			(at 34.925 172.72 0)
+			(at 37.465 185.42 0)
 			(effects
 				(font
@@
 		)
 		(property "Footprint" "Connector_PinHeader_2.54mm:PinHeader_1x04_P2.54mm_Vertical"
-			(at 34.29 177.8 0)
+			(at 36.83 180.34 0)
 			(effects
 				(font
@@
 		)
 		(property "Datasheet" "~"
-			(at 34.29 177.8 0)
+			(at 36.83 180.34 0)
 			(effects
 				(font
@@
 		)
 		(property "Description" "Generic connector, single row, 01x04, script generated"
-			(at 34.29 177.8 0)
+			(at 36.83 180.34 0)
 			(effects
 				(font
@@
 		)
 		(property "LCSC" ""
-			(at 34.29 177.8 0)
+			(at 36.83 180.34 0)
 			(effects
 				(font
@@
 	(symbol
 		(lib_id "power:+5V")
-		(at 53.34 187.96 0)
+		(at 90.17 168.91 0)
+		(mirror y)
 		(unit 1)
 		(exclude_from_sim no)
@@
 		(fields_autoplaced yes)
 		(property "Reference" "#PWR03"
-			(at 53.34 191.77 0)
+			(at 90.17 172.72 0)
 			(effects
 				(font
@@
 		)
 		(property "Value" "+5V"
-			(at 53.34 182.88 0)
+			(at 87.63 167.6399 0)
 			(effects
 				(font
 					(size 1.27 1.27)
 				)
+				(justify left)
 			)
 		)
 		(property "Footprint" ""
-			(at 53.34 187.96 0)
+			(at 90.17 168.91 0)
 			(effects
 				(font
@@
 		)
 		(property "Datasheet" ""
-			(at 53.34 187.96 0)
+			(at 90.17 168.91 0)
 			(effects
 				(font
@@
 		)
 		(property "Description" "Power symbol creates a global label with name \"+5V\""
-			(at 53.34 187.96 0)
+			(at 90.17 168.91 0)
 			(effects
 				(font
@@
 	(symbol
 		(lib_id "power:GND1")
-		(at 49.53 168.91 0)
+		(at 82.55 190.5 0)
+		(mirror y)
 		(unit 1)
 		(exclude_from_sim no)
@@
 		(fields_autoplaced yes)
 		(property "Reference" "#PWR05"
-			(at 49.53 175.26 0)
+			(at 82.55 196.85 0)
 			(effects
 				(font
@@
 		)
 		(property "Value" "GND1"
-			(at 49.53 173.99 0)
+			(at 80.01 191.7699 0)
 			(effects
 				(font
 					(size 1.27 1.27)
 				)
+				(justify left)
 			)
 		)
 		(property "Footprint" ""
-			(at 49.53 168.91 0)
+			(at 82.55 190.5 0)
 			(effects
 				(font
@@
 		)
 		(property "Datasheet" ""
-			(at 49.53 168.91 0)
+			(at 82.55 190.5 0)
 			(effects
 				(font
@@
 		)
 		(property "Description" "Power symbol creates a global label with name \"GND1\" , ground"
-			(at 49.53 168.91 0)
+			(at 82.55 190.5 0)
 			(effects
 				(font
@@
 	(symbol
 		(lib_id "power:+3V3")
-		(at 63.5 180.34 0)
+		(at 90.17 177.8 0)
+		(mirror y)
 		(unit 1)
 		(exclude_from_sim no)
@@
 		(dnp no)
 		(property "Reference" "#PWR04"
-			(at 63.5 184.15 0)
+			(at 90.17 181.61 0)
 			(effects
 				(font
@@
 		)
 		(property "Value" "+3V3"
-			(at 63.754 181.356 0)
+			(at 89.916 178.816 0)
 			(effects
 				(font
@@
 		)
 		(property "Footprint" ""
-			(at 63.5 180.34 0)
+			(at 90.17 177.8 0)
 			(effects
 				(font
@@
 		)
 		(property "Datasheet" ""
-			(at 63.5 180.34 0)
+			(at 90.17 177.8 0)
 			(effects
 				(font
@@
 		)
 		(property "Description" "Power symbol creates a global label with name \"+3V3\""
-			(at 63.5 180.34 0)
+			(at 90.17 177.8 0)
 			(effects
 				(font
@@
 		(on_board yes)
 		(dnp no)
-		(fields_autoplaced yes)
 		(property "Reference" "#PWR019"
 			(at 67.31 168.91 0)
@@
 		)
 		(property "Value" "GND1"
-			(at 67.31 167.64 0)
+			(at 70.612 161.544 0)
 			(effects
 				(font
